Commit message: - stl updated - excess -stl's removed - xacro split into gripper and fingers - urdf.xacro updated - rviz config created - launch file created

File: ros2_control/onrobot_2fg7.ros2_control.xacro (robot description, xacro)
@@ -1,14 +1,9 @@
 <?xml version="1.0"?>
 <robot xmlns:xacro="http://www.ros.org/wiki/xacro">
-  <xacro:macro name="joint_hw" params="joint_num prefix">
-    <joint name="${prefix}joint_${joint_num}">
-      <state_interface name="position"/>
-    </joint>
-  </xacro:macro>
   <xacro:macro name="onrobot_2fg7_ros2_control" params="name prefix port address use_mock_hardware">
     <ros2_control name="${name}" type="system">
       <hardware>
         <xacro:unless value="${use_mock_hardware}">
-          <!-- <plugin>allegro_robot_driver/AllegroEffortHardwareInterface</plugin> -->
+          <plugin>onrobot_robot_driver/2fg7HardwareInterface</plugin>
           <param name="port">${port}</param>
           <param name="address">${address}</param>
@@ -19,5 +14,8 @@
         </xacro:if>
       </hardware>
-      <xacro:joint_hw joint_num="0" prefix="${prefix}"/>
+      <joint name="${prefix}">
+        <state_interface name="position"/>
+        <state_interface name="velocity"/>
+      </joint>
     </ros2_control>
   </xacro:macro>

File: urdf/onrobot_2fg7.urdf.xacro (robot description, xacro)
@@ -6,16 +6,18 @@
     <xacro:arg name="use_mock_hardware" default="false"/>
     <xacro:include filename="onrobot_2fg7.xacro"/>
-    <xacro:include filename="$(find onrobot_2FG7_gripper_description)/ros2_control/onrobot_2fg7.ros2_control.xacro"/>
+    <xacro:include filename="$(find onrobot_2fg7_description)/ros2_control/onrobot_2fg7.ros2_control.xacro"/>
     <link name="world"></link>
     <xacro:onrobot_2fg7 prefix="$(arg prefix)" parent="world">
         <origin xyz="0 0 0" rpy="0 0 0"/>
     </xacro:onrobot_2fg7>
+    <!-- Attach right fingertip -->
+    <xacro:onrobot_2fg7_fingertip prefix="right_" parent="$(arg prefix)right_attachment">
+        <origin xyz="0 0 0" rpy="0 0 3.14159265359"/>
+    </xacro:onrobot_2fg7_fingertip>
+    <!-- Attach left fingertip -->
+    <xacro:onrobot_2fg7_fingertip prefix="left_" parent="$(arg prefix)left_attachment">
+        <origin xyz="0 0 0" rpy="0 0 0"/>
+    </xacro:onrobot_2fg7_fingertip>
     <!-- ros2_control description -->
-    <xacro:allegro_ros2_control
-        name="onrobot_2fg7"
-        prefix="$(arg prefix)"
-        port="$(arg port)"
-        address="$(arg address)"
-        use_mock_hardware="$(arg use_mock_hardware)"
-        />
+    <xacro:onrobot_2fg7_ros2_control name="onrobot_2fg7" prefix="$(arg prefix)" port="$(arg port)" address="$(arg address)" use_mock_hardware="$(arg use_mock_hardware)" />
 </robot>

File: urdf/onrobot_2fg7.xacro (robot description, xacro)
@@ -1,8 +1,7 @@
 <?xml version="1.0" ?>
-<robot name="2fg7_outwards" xmlns:xacro="http://www.ros.org/wiki/xacro">
-<xacro:include filename="$(find onrobot_2fg7_description)/urdf/materials.xacro" />
-<xacro:macro name="onrobot_2fg7_gripper" params="prefix finger_configuration=outwards">
-  <xacro:property name="config" value="${finger_configuration}"/>
-  <xacro:if value="${config == 'outwards'}">
+<robot name="onrobot_2fg7"
+  xmlns:xacro="http://www.ros.org/wiki/xacro">
+  <xacro:include filename="$(find onrobot_2fg7_description)/urdf/materials.xacro" />
+  <xacro:macro name="onrobot_2fg7" params="prefix parent *origin">
     <link name="${prefix}base_link">
       <inertial>
@@ -25,25 +24,57 @@
       </collision>
     </link>
-    <link name="${prefix}right_finger_link">
+    <link name="${prefix}right_attachment"></link>
+    <link name="${prefix}left_attachment"></link>
+    <joint name="left_finger_joint" type="prismatic">
+      <origin xyz="0.0 0.0 0.12005" rpy="0 0 0"/>
+      <parent link="${prefix}base_link"/>
+      <child link="${prefix}left_attachment"/>
+      <axis xyz="-1.0 0.0 0.0"/>
+      <limit lower="0.0115" upper="0.0305" effort="140" velocity="0.45"/>
+      <!-- total 0.38 -->
+    </joint>
+    <joint name="right_finger_joint" type="prismatic">
+      <origin xyz="0.0 0.0 0.12005" rpy="0 0 0"/>
+      <parent link="${prefix}base_link"/>
+      <child link="${prefix}right_attachment"/>
+      <axis xyz="1.0 0.0 0.0"/>
+      <limit lower="-0.0115" upper="-0.0305" effort="140" velocity="0.45"/>
+      <mimic joint="left_finger_joint" multiplier="1.0"/>
+    </joint>
+    <joint name="${prefix}2fg7_attach_joint" type="fixed">
+      <parent link="${parent}"/>
+      <child link="${prefix}base_link"/>
+      <xacro:insert_block name="origin"/>
+      <axis xyz="0 0 1"/>
+    </joint>
+  </xacro:macro>
+  <xacro:macro name="onrobot_2fg7_fingertip" params="prefix parent *origin">
+    <link name="${prefix}onrobot_2fg7_finger_link">
       <inertial>
-        <origin xyz="0.017874296677847158 0.02949104051991925 0.01523421548622829" rpy="0 0 0"/>
+        <origin xyz="0.0 0.0 0.0" rpy="0 0 0"/>
         <mass value="0.023219383355922288"/>
         <inertia ixx="6e-06" iyy="5e-06" izz="2e-06" ixy="-0.0" iyz="-0.0" ixz="1e-06"/>
       </inertial>
       <visual>
-        <origin xyz="0.054361 0.029494 -0.12005" rpy="0 0 0"/>
+        <origin xyz="0.0 0.0 0.0" rpy="0 0 0"/>
         <geometry>
-          <mesh filename="package://onrobot_2fg7_description/meshes/right_finger_link.stl" scale="0.001 0.001 0.001"/>
+          <mesh filename="package://onrobot_2fg7_description/meshes/finger_link.stl" scale="0.001 0.001 0.001"/>
         </geometry>
         <material name="silver"/>
       </visual>
       <collision name="right_finger_collision">
-        <origin xyz="0.054361 0.029494 -0.12005" rpy="0 0 0"/>
+        <origin xyz="0.0 0.0 0.0" rpy="0 0 0"/>
         <geometry>
-          <mesh filename="package://onrobot_2fg7_description/meshes/right_finger_link.stl" scale="0.001 0.001 0.001"/>
+          <mesh filename="package://onrobot_2fg7_description/meshes/finger_link.stl" scale="0.001 0.001 0.001"/>
         </geometry>
       </collision>
     </link>
-    <link name="${prefix}left_finger_link">
+    <joint name="${prefix}onrobot_2fg7_fingertip_joint" type="fixed">
+      <parent link="${parent}"/>
+      <child link="${prefix}onrobot_2fg7_finger_link"/>
+      <xacro:insert_block name="origin"/>
+      <axis xyz="0 0 1"/>
+    </joint>
+    <!-- <link name="${prefix}left_finger_link">
       <inertial>
         <origin xyz="0.004247703322119739 0.029496959480080673 0.015234215486237948" rpy="0 0 0"/>
@@ -64,98 +95,5 @@
         </geometry>
       </collision>
-    </link>
-    <joint name="left_finger_joint" type="prismatic">
-      <origin xyz="0.032239 -0.029494 0.12005" rpy="0 0 0"/>
-      <parent link="${prefix}base_link"/>
-      <child link="${prefix}left_finger_link"/>
-      <axis xyz="-1.0 0.0 0.0"/>
-      <limit lower="0.0" upper="0.019" effort="140" velocity="0.45"/> <!-- total 0.38 -->
-    </joint>
-    <joint name="right_finger_joint" type="prismatic">
-      <origin xyz="-0.054361 -0.029494 0.12005" rpy="0 0 0"/>
-      <parent link="${prefix}base_link"/>
-      <child link="${prefix}right_finger_link"/>
-      <axis xyz="1.0 0.0 0.0"/>
-      <limit lower="-0.019" upper="0.019" effort="140" velocity="0.45"/>
-      <mimic joint="left_finger_joint" multiplier="1.0"/>
-    </joint>
-  </xacro:if>
-   <xacro:if value="${config == 'inwards'}">
-    <link name="${prefix}base_link">
-      <inertial>
-        <origin xyz="-4.8989159583623376e-05 2.847569602502098e-06 0.06811082379775064" rpy="0 0 0"/>
-        <mass value="1.2646523179240972"/>
-        <inertia ixx="0.001504" iyy="0.001812" izz="0.001053" ixy="-0.0" iyz="0.0" ixz="-3e-06"/>
-      </inertial>
-      <visual>
-        <origin xyz="0 0 0" rpy="0 0 0"/>
-        <geometry>
-          <mesh filename="package://onrobot_2fg7_description/meshes/base_link.stl" scale="0.001 0.001 0.001"/>
-        </geometry>
-        <material name="silver"/>
-      </visual>
-      <collision>
-        <origin xyz="0 0 0" rpy="0 0 0"/>
-        <geometry>
-          <mesh filename="package://onrobot_2fg7_description/meshes/base_link.stl" scale="0.001 0.001 0.001"/>
-        </geometry>
-      </collision>
-    </link>
-    <link name="${prefix}right_finger_link">
-      <inertial>
-        <origin xyz="0.029847703322119633 0.029496959480087837 0.015234215486232036" rpy="0 0 0"/>
-        <mass value="0.023219383355922288"/>
-        <inertia ixx="6e-06" iyy="5e-06" izz="2e-06" ixy="-0.0" iyz="0.0" ixz="-1e-06"/>
-      </inertial>
-      <visual>
-        <origin xyz="0.054361 0.029494 -0.12005" rpy="0 0 0"/>
-        <geometry>
-          <mesh filename="package://onrobot_2fg7_description/meshes/inwards/right_finger_link.stl" scale="0.001 0.001 0.001"/>
-        </geometry>
-        <material name="silver"/>
-      </visual>
-      <collision>
-        <origin xyz="0.054361 0.029494 -0.12005" rpy="0 0 0"/>
-        <geometry>
-          <mesh filename="package://onrobot_2fg7_description/meshes/inwards/right_finger_link.stl" scale="0.001 0.001 0.001"/>
-        </geometry>
-      </collision>
-    </link>
-    <link name="${prefix}left_finger_link">
-      <inertial>
-        <origin xyz="-0.007725703322151688 0.029491040519911117 0.015234215486238503" rpy="0 0 0"/>
-        <mass value="0.023219383355922288"/>
-        <inertia ixx="6e-06" iyy="5e-06" izz="2e-06" ixy="-0.0" iyz="-0.0" ixz="1e-06"/>
-      </inertial>
-      <visual>
-        <origin xyz="-0.032239 0.029494 -0.12005" rpy="0 0 0"/>
-        <geometry>
-          <mesh filename="package://onrobot_2fg7_description/meshes/inwards/left_finger_link.stl" scale="0.001 0.001 0.001"/>
-        </geometry>
-        <material name="silver"/>
-      </visual>
-      <collision>
-        <origin xyz="-0.032239 0.029494 -0.12005" rpy="0 0 0"/>
-        <geometry>
-          <mesh filename="package://onrobot_2fg7_description/meshes/inwards/left_finger_link.stl" scale="0.001 0.001 0.001"/>
-        </geometry>
-      </collision>
-    </link>
-    <joint name="left_finger_joint" type="prismatic">
-      <origin xyz="0.032239 -0.029494 0.12005" rpy="0 0 0"/>
-      <parent link="${prefix}base_link"/>
-      <child link="${prefix}left_finger_link"/>
-      <axis xyz="-1.0 0.0 0.0"/>
-      <limit upper="0.0" lower="0.019" effort="100" velocity="0.45"/>
-    </joint>
-    <joint name="right_finger_joint" type="prismatic">
-      <origin xyz="-0.054361 -0.029494 0.12005" rpy="0 0 0"/>
-      <parent link="${prefix}base_link"/>
-      <child link="${prefix}right_finger_link"/>
-      <axis xyz="1.0 0.0 0.0"/>
-      <limit lower="-0.019" upper="0.019" effort="100" velocity="0.45"/>
-      <mimic joint="left_finger_joint" multiplier="1.0"/>
-    </joint>
-   </xacro:if>
- </xacro:macro>
+    </link> -->
+  </xacro:macro>
 </robot>

Commit message: - package xml - removed unused deps - rviz launch - added args - control.xacro - added params - urdf.xacro - added args - xacro - added missing prefix, changed joint name

File: ros2_control/onrobot_2fg7.ros2_control.xacro (robot description, xacro)
@@ -1,11 +1,14 @@
 <?xml version="1.0"?>
 <robot xmlns:xacro="http://www.ros.org/wiki/xacro">
-  <xacro:macro name="onrobot_2fg7_ros2_control" params="name prefix port address use_mock_hardware">
+  <xacro:macro name="onrobot_2fg7_ros2_control" params="name prefix port address force position_filtering velocity_filtering use_mock_hardware">
     <ros2_control name="${name}" type="system">
       <hardware>
         <xacro:unless value="${use_mock_hardware}">
-          <plugin>onrobot_robot_driver/2fg7HardwareInterface</plugin>
+          <plugin>onrobot_robot_driver/Onrobot2FG7PositionHardwareInterface</plugin>
           <param name="port">${port}</param>
           <param name="address">${address}</param>
+          <param name="force">100</param>
+          <param name="position_filtering">1.0</param>
+          <param name="velocity_filtering">1.0</param>
         </xacro:unless>
         <xacro:if value="${use_mock_hardware}">
@@ -14,7 +17,8 @@
         </xacro:if>
       </hardware>
-      <joint name="${prefix}">
+      <joint name="${prefix}gripper_joint">
         <state_interface name="position"/>
         <state_interface name="velocity"/>
+        <command_interface name="position"/>
       </joint>
     </ros2_control>

File: urdf/onrobot_2fg7.urdf.xacro (robot description, xacro)
@@ -4,4 +4,7 @@
     <xacro:arg name="port" default="502" />
     <xacro:arg name="address" default="" />
+    <xacro:arg name="force" default="" />
+    <xacro:arg name="position_filtering" default="" />
+    <xacro:arg name="velocity_filtering" default="" />
     <xacro:arg name="use_mock_hardware" default="false"/>
     <xacro:include filename="onrobot_2fg7.xacro"/>
@@ -25,4 +28,7 @@
     port="$(arg port)"
     address="$(arg address)"
+    force="$(arg force)"
+    position_filtering="$(arg position_filtering)"
+    velocity_filtering="$(arg velocity_filtering)"
     use_mock_hardware="$(arg use_mock_hardware)" />
 </robot>

File: urdf/onrobot_2fg7.xacro (robot description, xacro)
@@ -26,5 +26,5 @@
     <link name="${prefix}right_attachment"></link>
     <link name="${prefix}left_attachment"></link>
-    <joint name="left_finger_joint" type="prismatic">
+    <joint name="${prefix}gripper_joint" type="prismatic">
       <origin xyz="0.0 0.0 0.12005" rpy="0 0 0"/>
       <parent link="${prefix}base_link"/>
@@ -34,5 +34,5 @@
       <!-- total 0.38 -->
     </joint>
-    <joint name="right_finger_joint" type="prismatic">
+    <joint name="${prefix}right_finger_joint" type="prismatic">
       <origin xyz="0.0 0.0 0.12005" rpy="0 0 0"/>
       <parent link="${prefix}base_link"/>
@@ -40,5 +40,5 @@
       <axis xyz="1.0 0.0 0.0"/>
       <limit lower="-0.0115" upper="-0.0305" effort="140" velocity="0.45"/>
-      <mimic joint="left_finger_joint" multiplier="1.0"/>
+      <mimic joint="${prefix}gripper_joint" multiplier="1.0"/>
     </joint>
     <joint name="${prefix}2fg7_attach_joint" type="fixed">

Commit message: Use commanded, comments

File: ros2_control/onrobot_2fg7.ros2_control.xacro (robot description, xacro)
@@ -11,4 +11,5 @@
           <param name="position_filtering">1.0</param>
           <param name="velocity_filtering">1.0</param>
+          <param name="use_commanded">true</param>
         </xacro:unless>
         <xacro:if value="${use_mock_hardware}">

File: urdf/onrobot_2fg7.xacro (robot description, xacro)
@@ -39,5 +39,5 @@
       <child link="${prefix}right_attachment"/>
       <axis xyz="1.0 0.0 0.0"/>
-      <limit lower="-0.0115" upper="-0.0305" effort="140" velocity="0.45"/>
+      <limit lower="0.0115" upper="0.0305" effort="140" velocity="0.45"/>
       <mimic joint="${prefix}gripper_joint" multiplier="1.0"/>
     </joint>
@@ -76,24 +76,4 @@
       <axis xyz="0 0 1"/>
     </joint>
-    <!-- <link name="${prefix}left_finger_link">
-      <inertial>
-        <origin xyz="0.004247703322119739 0.029496959480080673 0.015234215486237948" rpy="0 0 0"/>
-        <mass value="0.023219383355922288"/>
-        <inertia ixx="6e-06" iyy="5e-06" izz="2e-06" ixy="-0.0" iyz="0.0" ixz="-1e-06"/>
-      </inertial>
-      <visual>
-        <origin xyz="-0.032239 0.029494 -0.12005" rpy="0 0 0"/>
-        <geometry>
-          <mesh filename="package://onrobot_2fg7_description/meshes/left_finger_link.stl" scale="0.001 0.001 0.001"/>
-        </geometry>
-        <material name="silver"/>
-      </visual>
-      <collision name="left_finger_collision">
-        <origin xyz="-0.032239 0.029494 -0.12005" rpy="0 0 0"/>
-        <geometry>
-          <mesh filename="package://onrobot_2fg7_description/meshes/left_finger_link.stl" scale="0.001 0.001 0.001"/>
-        </geometry>
-      </collision>
-    </link> -->
   </xacro:macro>
 </robot>
